File: pcb/DivaConSliderMpr/DivaConSlider.kicad_sch (KiCad schematic)
At the start: 189 parts, among them J1 Slider I2C, J2 Slider LED, J3 Display I2C, J4 Display, U1 MPR121QR2, U2 MPR121QR2, U3 MPR121QR2, U4 MPR121QR2

Commit message: placing both I2C buses on the same connector
Parts:
- removed C1: 0.1uF, Capacitor_SMD:C_0805_2012Metric_Pad1.18x1.45mm_HandSolder, symbol Device:C_Small
- removed J1: Slider I2C, Connector_JST:JST_PH_B4B-PH-K_1x04_P2.00mm_Vertical, symbol Connector_Generic:Conn_01x04
- removed J3: Display I2C, Connector_JST:JST_PH_B4B-PH-K_1x04_P2.00mm_Vertical, symbol Connector_Generic:Conn_01x04
- removed J4: Display, Connector_PinHeader_2.54mm:PinHeader_1x04_P2.54mm_Vertical, symbol Connector_Generic:Conn_01x04
- removed R12, R3: 10k, Resistor_SMD:R_0805_2012Metric_Pad1.20x1.40mm_HandSolder, symbol Device:R
- removed R13: 470, Resistor_SMD:R_0805_2012Metric_Pad1.20x1.40mm_HandSolder, symbol Device:R
- removed U1: MPR121QR2, Package_DFN_QFN:UQFN-20_3x3mm_P0.4mm, symbol Sensor_Touch:MPR121QR2
- added C7: 100n, Capacitor_SMD:C_0805_2012Metric_Pad1.18x1.45mm_HandSolder, symbol Device:C_Small
- added J1: Conn_01x06, symbol Connector_Generic:Conn_01x06
- added R8: 75k, Resistor_SMD:R_0805_2012Metric_Pad1.20x1.40mm_HandSolder, symbol Device:R
- added U4: MPR121QR2, Package_DFN_QFN:UQFN-20_3x3mm_P0.4mm, symbol Sensor_Touch:MPR121QR2
- C1: renamed from C7; value 0.1uF -> 100n
- C10, C11, C12, C13, C14, C15, C16, C17, C18, C19, C20, C21, C22, C23, C24, C25, C26, C27, C28, C29, C30, C31, C32, C33, C34, C35, C36, C37, C38, C39, C40, C41, C42, C43, C44, C45, C46, C47, C48, C49, C50, C51, C52, C53, C54, C55, C56, C57, C58, C59, C60, C61, C62, C63, C64, C65, C66, C67, C68, C69, C70, C71, C72, C9: value 0.1uF -> 100n; footprint Capacitor_SMD:C_0805_2012Metric_Pad1.18x1.45mm_HandSolder -> (none)
- C2, C3, C4, C5, C6, C8: value 0.1uF -> 100n
- J2: value Slider LED -> Conn_01x04; footprint Connector_JST:JST_PH_B4B-PH-K_1x04_P2.00mm_Vertical -> (none)
- R1: value 10k -> 4k7
- R10, R9: value 10k -> 75k
- R11: value 10k -> 470R; footprint Resistor_SMD:R_0805_2012Metric_Pad1.20x1.40mm_HandSolder -> (none)
- R2: value 75k -> 4k7
- R4, R6: value 75k -> 10k
- renumbered H8 to H1, H14 to H10, H22 to H11, H30 to H12, H5 to H13, H13 to H14, H21 to H15, H29 to H16, H4 to H17, H12 to H18, H20 to H19, H16 to H2, H28 to H20, H3 to H21, H11 to H22, H19 to H23, H27 to H24, H2 to H25, H10 to H26, H18 to H27, H26 to H28, H1 to H29, H24 to H3, H9 to H30, H17 to H31, H25 to H32, H32 to H4, H7 to H5, H15 to H6, H23 to H7, H31 to H8, H6 to H9, R7 to R3, R8 to R7, U4 to U1
Connections:
- net Slider LED Data is gone; now on net I2C_SDA: J2.4 (Pin_4)
- net +3V3: now also C2.1, C4.1, J2.1 (Pin_1), R2.1, R3.2, R4.2, R5.2, R6.2, U3.4 (ADDR), J1.5 (Pin_5), U4.20 (VDD); no longer C5.1, R10.2, R3.1, R5.1, R9.2, U2.4 (ADDR)
- net +5V: now also C10.1, C11.1, C12.1, C13.1, C14.1, C15.1, C16.1, C17.1, C18.1, C19.1, C20.1, C21.1, C22.1, C23.1, C24.1, C25.1, C26.1, C27.1, C28.1, C29.1, C30.1, C31.1, C32.1, C33.1, C34.1, C35.1, C36.1, C37.1, C38.1, C39.1, C40.1, C41.1, C42.1, C43.1, C44.1, C45.1, C46.1, C47.1, C48.1, C49.1, C50.1, C51.1, C52.1, C53.1, C54.1, C55.1, C56.1, C57.1, C58.1, C59.1, C60.1, C61.1, C62.1, C63.1, C64.1, C65.1, C66.1, C67.1, C68.1, C69.1, C70.1, C71.1, C72.1, C9.1, J1.6 (Pin_6); no longer C10.2, C11.2, C12.2, C13.2, C14.2, C15.2, C16.2, C17.2, C18.2, C19.2, C20.2, C21.2, C22.2, C23.2, C24.2, C25.2, C26.2, C27.2, C28.2, C29.2, C30.2, C31.2, C32.2, C33.2, C34.2, C35.2, C36.2, C37.2, C38.2, C39.2, C40.2, C41.2, C42.2, C43.2, C44.2, C45.2, C46.2, C47.2, C48.2, C49.2, C50.2, C51.2, C52.2, C53.2, C54.2, C55.2, C56.2, C57.2, C58.2, C59.2, C60.2, C61.2, C62.2, C63.2, C64.2, C65.2, C66.2, C67.2, C68.2, C69.2, C70.2, C71.2, C72.2, C9.2, J2.2 (Pin_2)
- net GND: now also C10.2, C11.2, C12.2, C13.2, C14.2, C15.2, C16.2, C17.2, C18.2, C19.2, C2.2, C20.2, C21.2, C22.2, C23.2, C24.2, C25.2, C26.2, C27.2, C28.2, C29.2, C30.2, C31.2, C32.2, C33.2, C34.2, C35.2, C36.2, C37.2, C38.2, C39.2, C4.2, C40.2, C41.2, C42.2, C43.2, C44.2, C45.2, C46.2, C47.2, C48.2, C49.2, C50.2, C51.2, C52.2, C53.2, C54.2, C55.2, C56.2, C57.2, C58.2, C59.2, C6.2, C60.2, C61.2, C62.2, C63.2, C64.2, C65.2, C66.2, C67.2, C68.2, C69.2, C70.2, C71.2, C72.2, C8.2, C9.2, J2.2 (Pin_2), R10.2, R7.2, R9.2, C7.2, J1.4 (Pin_4), R8.2, U4.4 (ADDR), U4.6 (VSS); no longer C10.1, C11.1, C12.1, C13.1, C14.1, C15.1, C16.1, C17.1, C18.1, C19.1, C2.1, C20.1, C21.1, C22.1, C23.1, C24.1, C25.1, C26.1, C27.1, C28.1, C29.1, C30.1, C31.1, C32.1, C33.1, C34.1, C35.1, C36.1, C37.1, C38.1, C39.1, C4.1, C40.1, C41.1, C42.1, C43.1, C44.1, C45.1, C46.1, C47.1, C48.1, C49.1, C50.1, C51.1, C52.1, C53.1, C54.1, C55.1, C56.1, C57.1, C58.1, C59.1, C6.1, C60.1, C61.1, C62.1, C63.1, C64.1, C65.1, C66.1, C67.1, C68.1, C69.1, C70.1, C71.1, C72.1, C8.1, C9.1, J2.1 (Pin_1), R2.1, R4.1, R6.1, R7.1
- net at H24.1: now also U4.17 (LED5/ELE9)
- net at H30.1: now also U2.19 (LED7/ELE11); no longer U3.19 (LED7/ELE11)
- net at U2.1 (~{IRQ}): now also R4.1
- net at D3.3 (DOUT): now also D4.1 (DIN); no longer D2.1 (DIN)
- net at D2.3 (DOUT): now also D3.1 (DIN); no longer D1.1 (DIN)
- net at D32.1 (DIN): now also D31.3 (DOUT)
- net at D31.1 (DIN): now also D30.3 (DOUT); no longer D32.3 (DOUT)
- net at D33.1 (DIN): now also D32.3 (DOUT); no longer D1.3 (DOUT)
- net at D14.3 (DOUT): now also D15.1 (DIN); no longer D13.1 (DIN)
- net at D12.1 (DIN): now also D11.3 (DOUT); no longer D13.3 (DOUT)
- net at D5.3 (DOUT): now also D6.1 (DIN); no longer D4.1 (DIN)
- net at D4.3 (DOUT): now also D5.1 (DIN); no longer D3.1 (DIN)
- net at U3.7 (REXT): now also R9.1; no longer R6.2
- net at H14.1: now also U2.15 (LED3/ELE7); no longer U3.15 (LED3/ELE7)
- net at U1.5 (VREG): now also C5.1; no longer C8.2
- net at D19.3 (DOUT): now also D20.1 (DIN); no longer D18.1 (DIN)
- net at D17.1 (DIN): now also D16.3 (DOUT); no longer D18.3 (DOUT)
- net at D7.1 (DIN): now also D6.3 (DOUT); no longer D8.3 (DOUT)
- net at D7.3 (DOUT): now also D8.1 (DIN); no longer D6.1 (DIN)
- net at U2.7 (REXT): now also R8.1; no longer R4.2
- net at H4.1: now also U4.12 (LED0/ELE4)
- net at D12.3 (DOUT): now also D13.1 (DIN); no longer D11.1 (DIN)
- net at D9.3 (DOUT): now also D10.1 (DIN); no longer D8.1 (DIN)
- net at D10.3 (DOUT): now also D11.1 (DIN); no longer D9.1 (DIN)
- net at H11.1: now also U3.14 (LED2/ELE6); no longer U2.14 (LED2/ELE6)
- net at D22.1 (DIN): now also D21.3 (DOUT); no longer D23.3 (DOUT)
- net at D22.3 (DOUT): now also D23.1 (DIN); no longer D21.1 (DIN)
- net at U2.12 (LED0/ELE4): now also H2.1; no longer H3.1
- net at H7.1: now also U3.13 (LED1/ELE5); no longer U2.13 (LED1/ELE5)
- net at H15.1: now also U3.15 (LED3/ELE7); no longer U2.15 (LED3/ELE7)
- net at U2.16 (LED4/ELE8): now also H18.1; no longer H19.1
- net at H23.1: now also U3.17 (LED5/ELE9); no longer U2.17 (LED5/ELE9)
- net at H27.1: now also U3.18 (LED6/ELE10); no longer U2.18 (LED6/ELE10)
- net at H31.1: now also U3.19 (LED7/ELE11); no longer U2.19 (LED7/ELE11)
- net at U2.5 (VREG): now also C6.1; no longer C4.2
- net at H12.1: now also U4.14 (LED2/ELE6)
- net at D28.3 (DOUT): now also D29.1 (DIN); no longer D27.1 (DIN)
- net at D27.3 (DOUT): now also D28.1 (DIN); no longer D26.1 (DIN)
- net at U3.1 (~{IRQ}): now also R5.1; no longer R5.2
- net at U3.12 (LED0/ELE4): now also H3.1; no longer H2.1
- net I2C_SCL: now reaches R1.2
- net I2C_SCL: now also J2.3 (Pin_3), U1.2 (SCL), U1.4 (ADDR), U2.2 (SCL), J1.2 (Pin_2), U4.2 (SCL)
- net at D24.3 (DOUT): now also D25.1 (DIN); no longer D23.1 (DIN)
- net at U3.16 (LED4/ELE8): now also H19.1; no longer H18.1
- net I2C_SDA: now reaches R2.2
- net I2C_SDA: now also U1.3 (SDA), U2.3 (SDA), U2.4 (ADDR), U3.2 (SCL), U3.3 (SDA), J1.3 (Pin_3), U4.3 (SDA)
- net at U1.1 (~{IRQ}): now also R3.1; no longer R3.2
- net at D15.3 (DOUT): now also D16.1 (DIN); no longer D14.1 (DIN)
- net at H6.1: now also U2.13 (LED1/ELE5); no longer U3.13 (LED1/ELE5)
- net at H10.1: now also U2.14 (LED2/ELE6); no longer U3.14 (LED2/ELE6)
- net at H22.1: now also U2.17 (LED5/ELE9); no longer U3.17 (LED5/ELE9)
- net at H26.1: now also U2.18 (LED6/ELE10); no longer U3.18 (LED6/ELE10)
- net at U3.5 (VREG): now also C7.1; no longer C6.2
- net at H20.1: now also U4.16 (LED4/ELE8)
- net at D26.3 (DOUT): now also D27.1 (DIN); no longer D25.1 (DIN)
- net at D25.3 (DOUT): now also D26.1 (DIN); no longer D24.1 (DIN)
- net at U1.7 (REXT): now also R7.1; no longer R7.2
- net at D30.1 (DIN): now also D29.3 (DOUT); no longer D31.3 (DOUT)
- net at H8.1: now also U4.13 (LED1/ELE5)
- net at D20.3 (DOUT): now also D21.1 (DIN); no longer D19.1 (DIN)
- net at H32.1: now also U4.19 (LED7/ELE11)
- net at D17.3 (DOUT): now also D18.1 (DIN); no longer D16.1 (DIN)
- net at H28.1: now also U4.18 (LED6/ELE10)
- net at H16.1: now also U4.15 (LED3/ELE7)
- net +3V3_2 renamed LED_DATA
- net LED_DATA: now also J1.1 (Pin_1)
- net Display SCL: no longer names the net of R11.1
- net Display SCL: now also D1.1 (DIN)
- removed net Slider SCL: R9.1, U1.2 (SCL), U1.4 (ADDR), U2.2 (SCL), U3.2 (SCL)
- removed net Slider SDA: R10.1, U1.3 (SDA), U2.3 (SDA), U3.3 (SDA), U3.4 (ADDR)
- new net: R6.1, U4.1 (~{IRQ})
- new net: D13.3 (DOUT), D14.1 (DIN)
- new net: C8.1, U4.5 (VREG)
- new net: R10.1, U4.7 (REXT)
- new net: D1.3 (DOUT), D2.1 (DIN)
- new net: D8.3 (DOUT), D9.1 (DIN)
- new net: D23.3 (DOUT), D24.1 (DIN)
- new net: D18.3 (DOUT), D19.1 (DIN)
- no-connect marks 18 -> 21
Other:
- note added: "I2C Address: 0x5A"
- note added: "I2C Address: 0x5B"
- note added: "I2C Address: 0x5C"
- note added: "I2C Address: 0x5D"
- note removed: "0x5A"
- note removed: "0x5B"
- note removed: "0x5C"
- note removed: "0x5D"
- moved on the sheet: C1, H1, H10, H11, H12, H13, H14, H15, H16, H17, H18, H19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
