File: pcb/DivaConSlider/DivaConSlider.kicad_sch (KiCad schematic)
At the start: 229 parts, among them J1 HS96L03W2C03, J2 B8B-PH-SM4-TB, U1 MPR121QR2, U2 MPR121QR2, U3 MPR121QR2, U4 MPR121QR2, U5 74HCT1G14

Commit message: revision 1.1 pcb schematics and layout
Parts:
- renumbered C78 to C14, C14 to C15, C15 to C16, C16 to C17, C17 to C18, C18 to C19, C19 to C20, C20 to C21, C21 to C22, C22 to C23, C23 to C24, C24 to C25, C25 to C26, C26 to C27, C27 to C28, C28 to C29, C29 to C30, C30 to C31, C31 to C32, C32 to C33, C33 to C34, C34 to C35, C35 to C36, C36 to C37, C37 to C38, C38 to C39, C39 to C40, C40 to C41, C41 to C42, C42 to C43, C43 to C44, C44 to C45, C45 to C46, C46 to C47, C47 to C48, C48 to C49, C49 to C50, C50 to C51, C51 to C52, C52 to C53, C53 to C54, C54 to C55, C55 to C56, C56 to C57, C57 to C58, C58 to C59, C59 to C60, C60 to C61, C61 to C62, C62 to C63, C63 to C64, C64 to C65, C65 to C66, C66 to C67, C67 to C68, C68 to C69, C69 to C70, C70 to C71, C71 to C72, C72 to C73, C73 to C74, C74 to C75, C75 to C76, C76 to C77, C77 to C78, TP14 to TP1, TP1 to TP10, TP8 to TP11, TP9 to TP12, TP11 to TP13, TP5 to TP2, TP2 to TP3, TP3 to TP4, TP4 to TP5, TP7 to TP6, TP12 to TP7, TP6 to TP8, TP13 to TP9
Connections:
- net +3V3: now also J2.5 (Pin_5); no longer J2.7 (Pin_7)
- net +5V: now also J2.7 (Pin_7); no longer J2.8 (Pin_8)
- net DISPLAY_I2C_SCL: now also R1.2, R5.2; no longer R2.2, R8.2
- net DISPLAY_I2C_SDA: now also R2.2, R6.2; no longer R1.2, R7.2
- net GND: now also J2.6 (Pin_6); no longer J2.1 (Pin_1)
- net I2C_SCL: now also R7.2; no longer R5.2
- net I2C_SDA: now also R8.2; no longer R6.2
- net LED_DATA: now also J2.8 (Pin_8); no longer J2.6 (Pin_6)
- net at J2.2 (Pin_2): now also R6.1; no longer R8.1
- net at J2.4 (Pin_4): now also R8.1; no longer R6.1
- net at R5.1: now also J2.1 (Pin_1); no longer J2.5 (Pin_5)
Other:
- moved on the sheet: C6, C7, J2, R1, R2, R3, R4, R5, R6, R7, R8, TP10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

Commit message: Update PCBs to purchased revision
Main edit is using a ULN2003 NPN transistor array over discrete MOSFETs.
This was chosen because there was limited board space to put in
pull-down resistors on the board and it was complicating the single
layer routing. The PCB had to be expanded to 70x75mm anyways to
accommodate the SOIC ic anyways.

The schematics of the IO board were also updated to use net labels over
direct wiring. Due to the JST connectors and the Pi Pico schematic
symbol being mirrored, it was getting too difficult to have an
understandable schematic.

Minor edit was changing LED_DATA to nLED_DATA to signify that it is
an active low signal.
Parts:
- removed H41, H42, H43, H44, H45: Spacer_M3, MountingHole:MountingHole_3.2mm_M3_Pad, symbol Mechanical:MountingHole
- added H41, H42, H43, H44, H45: Standoff_M3, MountingHole:MountingHole_3.2mm_M3_Pad, symbol Mechanical:MountingHole_Pad
- added J3: 310-87-104-41-001101, Connector_PinHeader_2.54mm:PinHeader_1x04_P2.54mm_Vertical, symbol Connector_Generic:Conn_01x04
- added R17: 10k, Resistor_SMD:R_0603_1608Metric, symbol Device:R
- added SYM1: Logo_Open_Hardware_Small, Symbol:OSHW-Logo_5.7x6mm_SilkScreen, symbol Graphic:Logo_Open_Hardware_Small
- added SYM2: Leek, CustomLogos:Leek-Logo_6.3mm_Silkscreen, symbol CustomLogos:Leek
- added TP14: TestPoint, TestPoint:TestPoint_Pad_D1.5mm, symbol Connector:TestPoint
- C1, C10, C11, C14, C15, C16, C17, C18, C19, C2, C20, C21, C22, C23, C24, C25, C26, C27, C28, C29, C3, C30, C31, C32, C33, C34, C35, C36, C37, C38, C39, C4, C40, C41, C42, C43, C44, C45, C46, C47, C48, C49, C5, C50, C51, C52, C53, C54, C55, C56, C57, C58, C59, C60, C61, C62, C63, C64, C65, C66, C67, C68, C69, C70, C71, C72, C73, C74, C75, C76, C77, C78, C8, C9: Dielectric (none) -> X7R; Manufacturer (none) -> Samsung Electro-Mechanical; PartNumber (none) -> CL10B104KB8NNNC; Voltage (none) -> 50V
- C12, C6: footprint Capacitor_SMD:C_0603_1608Metric -> Capacitor_SMD:C_0805_2012Metric; Dielectric (none) -> X7R; Manufacturer (none) -> Samsung Electro-Mechanical; PartNumber (none) -> CL21B106KOQNNNE; Voltage (none) -> 16V
- C13, C7: Dielectric (none) -> X7R; Manufacturer (none) -> Samsung Electro-Mechanical; PartNumber (none) -> CL10B105KO8NNNC; Voltage (none) -> 16V
- D1, D10, D11, D12, D13, D14, D15, D16, D17, D18, D19, D2, D20, D21, D22, D23, D24, D25, D26, D27, D28, D29, D3, D30, D31, D32, D33, D34, D35, D36, D37, D38, D39, D4, D40, D41, D42, D43, D44, D45, D46, D47, D48, D49, D5, D50, D51, D52, D53, D54, D55, D56, D57, D58, D59, D6, D60, D61, D62, D63, D64, D7, D8, D9: Manufacturer (none) -> OPSCO Electronics; PartNumber (none) -> SK6812SIDE-A
- H1, H2, H3, H4: value Spacer_M2 -> Standoff_M2; footprint (none) -> MountingHole:MountingHole_2.2mm_M2_Pad
- H37, H38, H39, H40: value Spacer_M3 -> Standoff_M3
- J1: Manufacturer (none) -> Hansheng; PartNumber (none) -> HS96L03W2C03
- J2: value B8B-PH-SM4-TB -> B8B-PH-SM4-TBT; Manufacturer (none) -> JST; PartNumber (none) -> B8B-PH-SM4-TBT
- R1, R2, R3, R4: Manufacturer (none) -> Stackpole Electronics; PartNumber (none) -> RMCF0603FT4K70
- R10, R11, R12, R9: Manufacturer (none) -> Stackpole Electronics; PartNumber (none) -> RMCF0603FT10K0
- R13, R14, R15, R16: Manufacturer (none) -> Stackpole Electronics; PartNumber (none) -> RMCF0603FT75K0
- R18: renamed from R17; Manufacturer (none) -> Stackpole Electronics; PartNumber (none) -> RMCF0603FT470R
- R5, R6, R7, R8: Manufacturer (none) -> Stackpole Electronics; PartNumber (none) -> RMCF0603ZT0R00
- TP1, TP10, TP11, TP12, TP13, TP6, TP7, TP8, TP9: now left out of the parts list
- TP2: renamed from TP4; now left out of the parts list
- TP3: renamed from TP5; now left out of the parts list
- TP4: renamed from TP2; now left out of the parts list
- TP5: renamed from TP3; now left out of the parts list
- U1, U2, U3, U4: Manufacturer (none) -> Nexperia; PartNumber (none) -> MPR121QR2
- U5: value 74HCT1G14 -> 74HCT1G14GV,125; Manufacturer (none) -> Nexperia; PartNumber (none) -> 74HCT1G14GV,125
- renumbered R18 to R19
Connections:
- net +3V3: now also R10.1, R11.1, R9.1, TP14.1; no longer R10.2, R11.2, R9.2
- net +5V: now also R17.2
- net at U1.1 (~{IRQ}): now also R9.2; no longer R9.1
- net at U3.1 (~{IRQ}): now also R11.2; no longer R11.1
- net at U2.1 (~{IRQ}): now also R10.2; no longer R10.1
- net LED_DATA renamed nLED_DATA
- net nLED_DATA: now also R17.1
- no-connect marks 16 -> 25
Other:
- moved on the sheet: C1, C12, C13, C6, C7, FID1, FID2, FID3, FID4, J1, J2, R1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
